File: Eagle/millefori/MILLEFORI.brd (EAGLE design)
At the start: 72.7 x 47 mm, 18 parts

Commit message: eagle2
Parts:
- removed A7: (no value), SparkFun-Connectors:1X01
- removed R3, R4: 1k, SparkFun-Resistors:AXIAL-0.3EZ
- moved +5V 2.54 mm to (53.3, 15.2)
Connections:
- removed net A7: A7.1, R3.P$1, R4.P$2
- net GND: no longer R4.P$1
- net VIN: no longer R3.P$2
Routing:
- net A0: track 57.8 -> 47.6 mm
- net A7: track 5.08 -> 0.00 mm
- net VIN: track 88.8 -> 84.7 mm, vias 4 -> 3
- net GND: track 172.2 -> 169.7 mm
Other:
- board text removed: "A0"
Changed lines of the file:
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@@
 <text x="27.94" y="29.21" size="1.778" layer="27" rot="R270" align="center-left">D11</text>
 <text x="69.215" y="8.89" size="1.778" layer="27" rot="R180" align="center-left">GND</text>
-<text x="62.23" y="15.24" size="1.778" layer="27" align="center-left">VIN</text>
-<text x="67.31" y="30.48" size="1.778" layer="27" align="center-left">5V</text>
+<text x="39.37" y="21.59" size="1.778" layer="27" align="center-left">VIN</text>
+<text x="62.23" y="24.13" size="1.778" layer="27" rot="R180" align="center-left">5V</text>
 <text x="34.29" y="15.24" size="1.778" layer="27" align="center-left">A7</text>
-<text x="52.07" y="15.24" size="1.778" layer="27" rot="R180" align="center-left">A0</text>
-<text x="54.61" y="11.43" size="1.778" layer="27" rot="R180" align="center-left">5V</text>
+<text x="52.07" y="11.43" size="1.778" layer="27" rot="R180" align="center-left">5V</text>
 <text x="40.64" y="30.48" size="1.778" layer="27" rot="R180" align="center-left">VIN</text>
 <text x="24.13" y="7.62" size="1.778" layer="27" rot="R180" align="center-left">GND</text>
 <text x="24.13" y="10.16" size="1.778" layer="27" rot="R180" align="center-left">5V</text>
 <text x="31.115" y="36.83" size="1.778" layer="27" rot="R180" align="center-left">GND</text>
-<text x="51.435" y="36.83" size="1.778" layer="27" rot="R180" align="center-left">GND</text>
+<text x="71.12" y="25.4" size="1.778" layer="27" align="center-left">GND</text>
 <text x="61.595" y="36.83" size="1.778" layer="27" rot="R180" align="center-left">GND</text>
 <text x="69.85" y="39.37" size="1.778" layer="27" rot="R180" align="center-left">VIN</text>
+<circle x="22.86" y="15.24" radius="0.635" width="0.3048" layer="21"/>
+<circle x="22.86" y="30.48" radius="0.635" width="0.3048" layer="21"/>
+<circle x="63.5" y="30.48" radius="0.635" width="0.3048" layer="21"/>
+<circle x="63.5" y="15.24" radius="0.635" width="0.3048" layer="21"/>
 </plain>
 <attributes>
@@
 </element>
 <element name="VIN0" library="SparkFun-Connectors" package="1X01" value="" x="60.96" y="15.24" rot="R270"/>
-<element name="+5V" library="SparkFun-Connectors" package="1X01" value="" x="55.88" y="15.24" rot="R270"/>
+<element name="+5V" library="SparkFun-Connectors" package="1X01" value="" x="53.34" y="15.24" rot="R270"/>
 <element name="JP2" library="SparkFun-Connectors" package="1X02" value="" x="58.42" y="30.48"/>
 <element name="JP1" library="SparkFun-Connectors" package="1X04" value="" x="50.8" y="30.48" rot="R180"/>
@@
 <element name="D13" library="SparkFun-Connectors" package="1X01" value="" x="25.4" y="15.24" rot="R180"/>
 <element name="U$3" library="18650" package="BATTERY_PACK_18650" value="18650" x="45.72" y="22.86"/>
-<element name="R3" library="SparkFun-Resistors" package="AXIAL-0.3EZ" value="1k" x="57.15" y="17.78">
-<attribute name="PROD_ID" value="RES-08380" x="57.15" y="17.78" size="1.778" layer="27" display="off"/>
-</element>
-<element name="R4" library="SparkFun-Resistors" package="AXIAL-0.3EZ" value="1k" x="53.34" y="24.13" rot="R270">
-<attribute name="PROD_ID" value="RES-08380" x="53.34" y="24.13" size="1.778" layer="27" rot="R270" display="off"/>
-</element>
-<element name="A7" library="SparkFun-Connectors" package="1X01" value="" x="53.34" y="15.24" rot="R180"/>
 <element name="A0" library="SparkFun-Connectors" package="1X01" value="" x="33.02" y="15.24" rot="R180"/>
 <element name="SERVO" library="SparkFun-Connectors" package="1X03" value="" x="25.4" y="12.7" rot="R270"/>
@@
 <wire x1="25.4" y1="10.16" x2="27.94" y2="10.16" width="1.27" layer="16"/>
 <via x="27.94" y="10.16" extent="1-16" drill="1.4" diameter="1.27" shape="square"/>
-<via x="55.88" y="12.7" extent="1-16" drill="1.4" diameter="1.27" shape="square"/>
+<via x="53.34" y="12.7" extent="1-16" drill="1.4" diameter="1.27" shape="square"/>
 <via x="63.5" y="22.86" extent="1-16" drill="1.4" diameter="1.27" shape="square"/>
-<wire x1="55.88" y1="15.24" x2="55.88" y2="12.7" width="1.27" layer="16"/>
-<wire x1="55.88" y1="20.32" x2="55.88" y2="15.24" width="1.27" layer="16"/>
-<wire x1="27.94" y1="10.16" x2="53.34" y2="10.16" width="0.3048" layer="1"/>
-<wire x1="53.34" y1="10.16" x2="55.88" y2="12.7" width="0.3048" layer="1" curve="90"/>
-<via x="55.88" y="20.32" extent="1-16" drill="1.4" diameter="1.27" shape="square"/>
+<wire x1="53.34" y1="15.24" x2="53.34" y2="12.7" width="1.27" layer="16"/>
+<wire x1="53.34" y1="17.78" x2="53.34" y2="15.24" width="1.27" layer="16"/>
+<wire x1="27.94" y1="10.16" x2="50.8" y2="10.16" width="0.3048" layer="1"/>
+<wire x1="50.8" y1="10.16" x2="53.34" y2="12.7" width="0.3048" layer="1" curve="90"/>
+<via x="53.34" y="17.78" extent="1-16" drill="1.4" diameter="1.27" shape="square"/>
 <wire x1="63.5" y1="22.86" x2="66.04" y2="22.86" width="1.27" layer="16"/>
-<wire x1="63.5" y1="22.86" x2="58.42" y2="22.86" width="0.3048" layer="1"/>
-<wire x1="58.42" y1="22.86" x2="55.88" y2="20.32" width="0.3048" layer="1" curve="90"/>
+<wire x1="63.5" y1="22.86" x2="55.88" y2="22.86" width="0.3048" layer="1"/>
+<wire x1="53.34" y1="17.78" x2="53.34" y2="20.32" width="0.3048" layer="1"/>
+<wire x1="53.34" y1="20.32" x2="55.88" y2="22.86" width="0.3048" layer="1" curve="-90"/>
 </signal>
 <signal name="VIN">
@@
 <contactref element="LEFT_M" pad="6"/>
 <contactref element="RIGHT_M" pad="6"/>
-<contactref element="R3" pad="P$2"/>
 <contactref element="S1" pad="2"/>
 <contactref element="S1" pad="1"/>
-<via x="60.96" y="12.7" extent="1-16" drill="1.4" diameter="1.27" shape="square"/>
+<via x="60.96" y="17.78" extent="1-16" drill="1.4" diameter="1.27" shape="square"/>
 <via x="38.1" y="33.02" extent="1-16" drill="1.4" diameter="1.27" shape="square"/>
 <wire x1="38.1" y1="33.02" x2="40.64" y2="33.02" width="1.27" layer="16"/>
-<wire x1="60.96" y1="17.78" x2="60.96" y2="15.24" width="1.27" layer="16"/>
 <wire x1="38.1" y1="33.02" x2="35.56" y2="33.02" width="1.27" layer="16"/>
-<wire x1="60.96" y1="15.24" x2="60.96" y2="12.7" width="1.27" layer="16"/>
-<wire x1="38.1" y1="33.02" x2="38.1" y2="35.56" width="0.3048" layer="1"/>
-<wire x1="60.96" y1="17.78" x2="73.66" y2="17.78" width="0.3048" layer="1"/>
-<wire x1="73.66" y1="17.78" x2="76.2" y2="20.32" width="0.3048" layer="1" curve="90"/>
-<wire x1="76.2" y1="20.32" x2="76.2" y2="38.1" width="0.3048" layer="1"/>
-<via x="76.2" y="38.1" extent="1-16" drill="1.4" diameter="2.54" shape="square"/>
+<wire x1="60.96" y1="15.24" x2="60.96" y2="17.78" width="1.27" layer="16"/>
+<wire x1="38.1" y1="33.02" x2="38.1" y2="35.56" width="0.6096" layer="1"/>
 <via x="71.12" y="38.1" extent="1-16" drill="1.4" diameter="1.27" shape="square"/>
-<wire x1="38.1" y1="35.56" x2="40.64" y2="38.1" width="0.3048" layer="1" curve="-90"/>
-<wire x1="40.64" y1="38.1" x2="71.12" y2="38.1" width="0.3048" layer="1"/>
+<wire x1="38.1" y1="35.56" x2="40.64" y2="38.1" width="0.6096" layer="1" curve="-90"/>
+<wire x1="40.64" y1="38.1" x2="71.12" y2="38.1" width="0.6096" layer="1"/>
 <wire x1="71.12" y1="38.1" x2="73.4822" y2="38.1" width="1.27" layer="16"/>
 <wire x1="73.4822" y1="38.1" x2="73.66" y2="38.2778" width="1.27" layer="16" curve="90"/>
-<wire x1="76.2" y1="38.1" x2="73.8378" y2="38.1" width="1.27" layer="16"/>
-<wire x1="73.8378" y1="38.1" x2="73.66" y2="38.2778" width="1.27" layer="16" curve="-90"/>
 <wire x1="73.66" y1="35.56" x2="73.66" y2="38.2778" width="1.27" layer="16"/>
+<wire x1="60.96" y1="17.78" x2="58.42" y2="20.32" width="0.6096" layer="1" curve="90"/>
+<wire x1="58.42" y1="20.32" x2="40.64" y2="20.32" width="0.6096" layer="1"/>
+<wire x1="40.64" y1="20.32" x2="38.1" y2="22.86" width="0.6096" layer="1" curve="-90"/>
+<wire x1="38.1" y1="22.86" x2="38.1" y2="33.02" width="0.6096" layer="1"/>
 </signal>
 <signal name="D0/RX">
@@
 <contactref element="U$3" pad="+3.7V_2"/>
 <contactref element="A0" pad="1"/>
-<wire x1="9.02" y1="32.36" x2="9.02" y2="13.36" width="1.27" layer="1"/>
-<via x="33.02" y="12.7" extent="1-16" drill="1.4" diameter="1.27" shape="square"/>
-<wire x1="33.02" y1="15.24" x2="33.02" y2="12.7" width="1.27" layer="16"/>
-<wire x1="33.02" y1="12.7" x2="33.02" y2="7.62" width="0.4064" layer="1"/>
-<wire x1="33.02" y1="7.62" x2="30.48" y2="5.08" width="0.4064" layer="1" curve="-90"/>
-<wire x1="30.48" y1="5.08" x2="12.7" y2="5.08" width="0.4064" layer="1"/>
-<wire x1="12.7" y1="5.08" x2="9.02" y2="8.76" width="0.4064" layer="1" curve="-90"/>
-<wire x1="9.02" y1="8.76" x2="9.02" y2="13.36" width="0.4064" layer="1"/>
-</signal>
-<signal name="A7">
-<contactref element="A7" pad="1"/>
-<contactref element="R3" pad="P$1"/>
-<contactref element="R4" pad="P$2"/>
-<wire x1="53.34" y1="20.32" x2="53.34" y2="17.78" width="1.27" layer="16"/>
-<wire x1="53.34" y1="17.78" x2="53.34" y2="15.24" width="1.27" layer="16"/>
+<wire x1="9.02" y1="32.36" x2="9.02" y2="22.86" width="1.27" layer="1"/>
+<via x="33.02" y="17.78" extent="1-16" drill="1.4" diameter="1.27" shape="square"/>
+<wire x1="9.02" y1="22.86" x2="9.02" y2="13.36" width="1.27" layer="1"/>
+<wire x1="33.02" y1="15.24" x2="33.02" y2="17.78" width="1.27" layer="16"/>
+<wire x1="30.48" y1="20.32" x2="11.56" y2="20.32" width="0.6096" layer="1"/>
+<wire x1="30.48" y1="20.32" x2="33.02" y2="17.78" width="0.6096" layer="1" curve="-90"/>
+<wire x1="11.56" y1="20.32" x2="9.02" y2="22.86" width="0.4064" layer="1" curve="-90"/>
 </signal>
 <signal name="+7,2V">
@@
 <contactref element="RIGHT_M" pad="1"/>
 <contactref element="U$3" pad="GND_2"/>
-<contactref element="R4" pad="P$1"/>
 <contactref element="SERVO" pad="3"/>
 <via x="71.12" y="7.62" extent="1-16" drill="1.4" diameter="1.27" shape="square"/>
@@
 <wire x1="66.04" y1="25.4" x2="68.58" y2="25.4" width="1.27" layer="16"/>
 <via x="68.58" y="25.4" extent="1-16" drill="1.4" diameter="1.27" shape="square"/>
-<wire x1="53.34" y1="30.48" x2="53.34" y2="27.94" width="1.27" layer="16"/>
 <wire x1="68.58" y1="25.4" x2="71.12" y2="22.86" width="0.3048" layer="1" curve="-90"/>
 <wire x1="71.12" y1="22.86" x2="71.12" y2="15.24" width="0.3048" layer="1"/>
